File: PCB/My-Hackpad.kicad_pcb (KiCad board)
At the start: 2 copper layers, 92.5 x 61.5 mm, 23 parts, among them J1 Display, SW1 SW_Push, SW2 SW_Push, SW3 SW_Push, SW4 SW_Push, SW5 SW_Push, SW6 SW_Push, SW7 RotaryEncoder_Switch, U1 MOUDLE-SEEEDUINO-XIAO

Commit message: production and stuff
Parts:
- added G***: LOGO, LOGO, F.Cu at (146.1, 82.0)
- added G***: LOGO, LOGO, F.Cu at (143.6, 106.4)
